File: MainBoard_Unlimited26/MainBoard_Unlimited26B/MainBoard_Unlimited26B.kicad_sch (KiCad schematic)
At the start: 48 parts, among them J1 power, J2 Conn_01x03_Pin, U1 TA6586, U10 TA6586, U2 TA6586, U3 TA6586, U4 TA6586, U5 TA6586, U7 ZC323000, U8 MP1584_3A_Mini

Commit message: REV ALL
Parts:
- removed C2: 1000uF, Capacitor_THT:CP_Radial_D10.0mm_P5.00mm, symbol Device:C_Polarized_Small
- removed D1, D10, D2, D3, D4, D5, D6, D7, D8, D9: D_Schottky, Diode_SMD:D_SMA, symbol Device:D_Schottky
- removed F1, F2, F3, F4, F5: Polyfuse, Fuse:Fuse_Bourns_MF-RG300, symbol Device:Polyfuse
- removed M5: (no value), Connector_JST:JST_XH_S2B-XH-A-1_1x02_P2.50mm_Horizontal, symbol Connector:Conn_01x02_Pin
- removed U1, U2, U3, U4, U5: TA6586, TA6586:TA6586-FOOTPRINT, symbol TA6586:TA6586
- added C13: 0.1uF, Capacitor_SMD:C_0805_2012Metric_Pad1.18x1.45mm_HandSolder, symbol Device:C_Small
- added C14: 1000uF, Capacitor_THT:CP_Radial_D10.0mm_P5.00mm, symbol Device:C_Polarized_Small
- added C2: 10uF, Capacitor_SMD:C_0805_2012Metric_Pad1.18x1.45mm_HandSolder, symbol Device:C_Small
- added J3, J4, L0: (no value), Connector_JST:JST_XH_B2B-XH-A_1x02_P2.50mm_Vertical, symbol Connector:Conn_01x02_Pin
- added J5: Conn_01x05_Pin, Connector_PinHeader_2.54mm:PinHeader_1x05_P2.54mm_Vertical, symbol Connector:Conn_01x05_Pin
- added J6: vreff mode, Connector_PinHeader_2.54mm:PinHeader_1x03_P2.54mm_Vertical, symbol Connector:Conn_01x03_Pin
- added J7: power, TerminalBlock:TerminalBlock_MaiXu_MX126-5.0-02P_1x02_P5.00mm, symbol Connector:Screw_Terminal_01x02
- added J8, J9: mconn, Connector_JST:JST_XH_B10B-XH-A_1x10_P2.50mm_Vertical, symbol Connector:Conn_01x10_Pin
- added Q1: BC846, Package_TO_SOT_SMD:SOT-23, symbol Transistor_BJT:BC846
- added R1: 10k, Resistor_SMD:R_0805_2012Metric_Pad1.20x1.40mm_HandSolder, symbol Device:R_Small
- added R2: 6k8, Resistor_SMD:R_0805_2012Metric_Pad1.20x1.40mm_HandSolder, symbol Device:R_Small
- added R3, R4, R5, R6: 0.1, Resistor_SMD:R_2512_6332Metric_Pad1.40x3.35mm_HandSolder, symbol Device:R_Small
- added R7: 4k7, Resistor_SMD:R_0805_2012Metric_Pad1.20x1.40mm_HandSolder, symbol Device:R_Small
- added U1: AMS1117-5.0, Package_TO_SOT_SMD:SOT-223-3_TabPin2, symbol Regulator_Linear:AMS1117-5.0
- added U2, U3, U4, U5: A4950E, Package_SO:SOIC-8-1EP_3.9x4.9mm_P1.27mm_EP2.41x3.3mm, symbol Driver_Motor:A4950E
- C11: value 0.1uF -> 10uF
- C6, C7, C8, C9: value 0.1uF -> 100nF
- J1: footprint terminal block right angel:TE_282815-2 -> TerminalBlock:TerminalBlock_MaiXu_MX126-5.0-02P_1x02_P5.00mm
- M1, M2, M3, M4, M6: footprint Connector_JST:JST_XH_S2B-XH-A-1_1x02_P2.50mm_Horizontal -> Connector_JST:JST_XH_B2B-XH-A_1x02_P2.50mm_Vertical
Connections:
- net +12V: now also C1.2, C3.2, C4.2, C5.2, C6.1, C7.1, C8.1, C9.1, C2.1, J7.1 (Pin_1), U1.3 (VI), U2.5 (VBB), U3.5 (VBB), U4.5 (VBB), U5.5 (VBB); no longer D13.2 (A), F7.1, J1.1 (Pin_1)
- net +5V: now also C13.1, L0.1 (Pin_1)
- net G: now also C1.1, C3.1, C4.1, C5.1, C13.2, C14.2, C2.2, J3.2 (Pin_2), J7.2 (Pin_2), J8.9 (Pin_9), J9.9 (Pin_9), Q1.2 (E), R2.1, R3.1, R4.1, R5.1, R6.1, U1.1 (GND), U2.1 (GND), U2.9 (PAD), U3.1 (GND), U3.9 (PAD), U4.1 (GND), U4.9 (PAD), U5.1 (GND), U5.9 (PAD); no longer C1.2, C3.2, C4.2, C5.2
- net PA0: now also J5.4 (Pin_4)
- net PA1: now also J5.5 (Pin_5)
- net PA10: now also J8.6 (Pin_6), J9.6 (Pin_6), U5.3 (IN1)
- net PA11: now also J8.5 (Pin_5), J9.5 (Pin_5), U5.2 (IN2)
- net PA8: now also J8.8 (Pin_8), J9.8 (Pin_8), U2.3 (IN1)
- net PA9: now also J8.7 (Pin_7), J9.7 (Pin_7), U2.2 (IN2)
- net PB6: now also J8.4 (Pin_4), J9.4 (Pin_4), U4.3 (IN1)
- net PB7: now also J8.3 (Pin_3), J9.3 (Pin_3), U4.2 (IN2)
- net PB8: now also J8.2 (Pin_2), J9.2 (Pin_2), U3.3 (IN1)
- net PB9: now also J8.1 (Pin_1), J9.1 (Pin_1), U3.2 (IN2)
- net DA5: now reaches U7.10 (A5)
- net PB10: now reaches U7.15 (B10)
- net PB10: now also J4.1 (Pin_1)
- net PB11: now reaches U7.16 (B11)
- net PB11: now also J4.2 (Pin_2)
- net R: now reaches U7.17 (R)
- net R: now also J3.1 (Pin_1)
- net PC13: now reaches U7.2 (C13)
- net PC13: now also J5.1 (Pin_1)
- net DB12: now reaches U7.21 (B12)
- net DB13: now reaches U7.22 (B13)
- net DB14: now reaches U7.23 (B14)
- net DB15: now reaches U7.24 (B15)
- net DB15: now also R7.1
- net PC14: now reaches U7.3 (C14)
- net PC14: now also J5.2 (Pin_2)
- net DB5: now reaches U7.33 (B5)
- net PC15: now reaches U7.4 (C15)
- net PC15: now also J5.3 (Pin_3)
- net DA4: now reaches U7.9 (A4)
- net at C11.1: now also R1.1, U1.2 (VO); no longer C5.1
- net at F6.1, U8.4 (VOUT+): now also C14.1
- net B1 renamed 1O2
- net 1O2: now also U3.8 (OUT2)
- net B2 renamed 2O2
- net 2O2: now also U4.8 (OUT2)
- net B3 renamed 3O2
- net 3O2: now also U5.8 (OUT2)
- net B4 renamed 4O2
- net 4O2: now also U2.8 (OUT2)
- net F1 renamed 1O1
- net 1O1: now also U3.6 (OUT1)
- net F2 renamed 2O1
- net 2O1: now also U4.6 (OUT1)
- net F3 renamed 3O1
- net 3O1: now also U5.6 (OUT1)
- net F4 renamed 4O1
- net 4O1: now also U2.6 (OUT1)
- new net: R4.2, U3.7 (LSS)
- new net: Q1.1 (B), R7.2
- new net: R5.2, U4.7 (LSS)
- new net: R6.2, U5.7 (LSS)
- new net: R3.2, U2.7 (LSS)
- new net: L0.2 (Pin_2), Q1.3 (C)
- new net +12Vs: D13.2 (A), F7.1, J1.1 (Pin_1)
- new net 2V: J6.1 (Pin_1), R1.2, R2.2
- new net REFF: J6.2 (Pin_2), U2.4 (VREF), U3.4 (VREF), U4.4 (VREF), U5.4 (VREF)
- new net Vreff: J6.3 (Pin_3), J8.10 (Pin_10), J9.10 (Pin_10)
- no-connect marks 1 -> 6
Other:
- moved on the sheet: C1, C10, C12, D11, D12, D13, F6, F7, J1, J2, M1, M2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
